File: pcb/AutoTuner.sch (EAGLE design)
At the start: 18 parts, among them IC1 TP4054-42-SOT25-R, J1 PJ324M, Q1 32,768kHz, U1 STM32F103C8T6, Y1 8MHz

Commit message: code init
Parts:
- removed J1: PJ324M, PJ324M:PJ324M
- added AUDIO_JACK: PJ324M, PJ324M:PJ324M
- added C10, C11: (no value), rcl:C-EUC0805
- added C12: 100n, rcl:C-EUC0805
- added C3, C5, C6: 10µ, rcl:C-EUC0805
- added C4: 0,1µ, rcl:C-EUC0805
- added C7: 10n, rcl:C-EUC0805
- added C8, C9: 20p, rcl:C-EUC0805
- added D1: MBR0520LT1G, Diode:SCHOTTKY_MBR0520LT1GDO-219
- added D2, D3, D4, D5, D6, D7: TESD5V0L1UC_RJG, TESD5V0L1UC_RJG:TESD5V0L1UC_RJG
- added DISPLAY: (no value), pinhead:PINHD-1X4
- added L1: 1,5µ, rcl:R-EU_R0805
- added LED1, LED2: (no value), led:LEDCHIPLED_0805
- added Q2: BSS123, Transistor:NMOSFET_BSS123_SOT23-GSD
- added Q3: BSS84, Transistor:PMOSFET_BSS84_SOT23-GSD
- added R10: 2M, rcl:R-EU_R0805
- added R11: (no value), rcl:R-EU_R0805
- added R12: 1M, rcl:R-EU_R0805
- added R13: 1k5, rcl:R-EU_R0805
- added R6: 1k66, rcl:R-EU_R0805
- added R7: 680, rcl:R-EU_R0805
- added R8: 10k, rcl:R-EU_R0805
- added R9: 800k, rcl:R-EU_R0805
- added USB-B: 61729-1011, Connector_USB:61729-1011
- C1: value (none) -> 100n
- Y1: LCSC C115962 -> (none); LCSC_PART (none) -> C115962
Connections:
- removed net N$4: C2.1, R2.1, RESET.NO
- new net AIN: C7.2, R10.2, R9.1
- new net JACK_L: AUDIO_JACK.RING_1
- new net JACK_R: AUDIO_JACK.TIP_2
- new net N$11: LED1.A, LED2.A, R7.2
- new net N$12: LED1.C, Q2.S
- new net N$15: U1.PA0_WKUP
- new net N$16: U1.PA1
- new net N$17: U1.PA2
- new net N$18: U1.PA3
- new net N$19: U1.PA4
- new net N$20: U1.PA5
- new net N$21: U1.PA6
- new net N$22: U1.PA7
- new net N$23: U1.PA8
- new net N$24: U1.PA9
- new net N$25: U1.PA10
- new net N$28: U1.PA15
- new net N$33: U1.PB0
- new net N$34: U1.PB1
- new net N$35: U1.PB2
- new net N$36: U1.PB3
- new net N$37: U1.PB4
- new net N$38: U1.PB5
- new net N$39: U1.PB6
- new net N$40: U1.PB7
- new net N$41: U1.PB8
- new net N$42: U1.PB9
- new net N$43: U1.PB10
- new net N$44: U1.PB11
- new net N$45: U1.PB12
- new net N$46: U1.PB13
- new net N$47: U1.PB14
- new net N$48: U1.PB15
- new net N$6: L1.1, PS1.L1
- new net N$7: L1.2, PS1.L2
- new net N$8: IC1.PROG, R6.2
- new net N$9: IC1.!CHRG, LED2.C, Q2.G, R8.2
- new net OSC32IN: C10.2, Q1.2, U1.PC14-OSC32_IN
- new net OSC32OUT: C11.2, Q1.1, U1.PC15-OSC32_OUT
- new net OSCIN: C8.2, R12.2, U1.PD0_OSC_IN, Y1.2
- new net OSCOUT: C9.2, R12.1, U1.PD1_OSC_OUT, Y1.1
- new net PC13: LED.A, U1.PC13-TAMPER-RTC
- new net RESET: C2.1, R2.1, RESET.NO, U1.NRST
- new net SWDCLK: D7.2, ST_LINK.2, U1.PA14
- new net SWDIO: D6.2, ST_LINK.3, U1.PA13
- new net VBAT: IC1.BAT, Q3.S, R9.2
- new net VBUS: C12.1, D1.A, D2.2, IC1.VCC, Q3.G, R11.2, R13.2, R7.1, R8.1, USB-B.VCC
- new net VIN: C3.1, D1.C, PS1.VIN, Q3.D
- net +3V3: now also C5.1, C6.1, D5.2, PS1.FB, PS1.VOUT, U1.VBAT, U1.VDD, U1.VDDA
- net BOOT0: now also U1.BOOT0
- net GND: now also AUDIO_JACK.SLEEVE, C10.1, C11.1, C12.2, C3.2, C4.2, C5.2, C6.2, C7.1, C8.1, C9.1, D2.1, D3.1, D4.1, D5.1, D6.1, D7.1, IC1.GND, PS1.GND, PS1.PGND, Q2.D, R10.1, R11.1, R6.1, U1.VSS, U1.VSSA, USB-B.GND, USB-B.SHIELD1, USB-B.SHIELD2
- net N$1: now also C4.1, PS1.EN, PS1.PS/SYNC, PS1.VINA; no longer LED.A
- net PA11: now also D3.2, U1.PA11, USB-B.D-; no longer ST_LINK.3
- net PA12: now also D4.2, R13.1, U1.PA12, USB-B.D+; no longer ST_LINK.2
Other:
- note added: "32kHz Quarz"
- note added: "8MHz Quarz"
- note added: "Battery Voltage Converter"
- note added: "Battery charger"
- note added: "Battery level"
- note added: "LEDs"
- note added: "Maximum voltage: 4.2 V * (2 M/(0.8 M+2 M)) = 3 V Maximum voltage: 3 V * (2 M/(0.8 M+2 M)) = 2,14 V Minimum voltage: 2.7 V * (2 M/(0.8 M+2 M)) = 1.93 V ADC value at 4.2 V – 12 bit setup: 3 V * (1/5) / 0.6 V * 4095 = 4095"
- note added: "Power IN"
- note added: "Voltage Source Selection"
- moved on the sheet: C1, C2, LED, POWER_LED, Q1, R1, R2, R3, R4, R5, RESET, S2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

Commit message: dcdc
Parts:
- added C20: 0.1u, rcl:C-EUC0805
- added C21, C24: 10u, rcl:CPOL-EU085CS-1AR
- added C22, C23: 1u, rcl:CPOL-EU085CS-1AR
- added D10, D11: 1N4002, diode:1N4004
- added D8, D9: 1N4004, diode:1N4004
- added IC2, IC3: LM317MBSTT3, v-reg:LM317MBSTT3
- added R14: 1.62M, rcl:R-EU_R0805
- added R15, R16: 100k, rcl:R-EU_R0805
- added R17: 394, rcl:R-EU_R0805
- added R18, R22: 240, rcl:R-EU_R0805
- added R21: 720, rcl:R-EU_R0805
- C3: value 10µ -> 2.2nF
- C4: value 0,1µ -> 47uF
- C5: value 10µ -> 10uF
- C6: value 10µ -> 0.1u
- L1: value 1,5µ -> 1.5uH
- PS1: value TPS63031DSKR -> TPS62147RGXR; device TPS63031DSKR:TPS63031DSKR -> TPS62147RGXR:TPS62147RGXR; LCSC_PART C15516 -> (none)
- R10: value 2M -> 2.5M
- R9: value 800k -> 10M
Connections:
- net AIN renamed A_BATTERY_LEVEL
- net JACK_L renamed N$4
- net JACK_R renamed AUDIO_IN
- new net +12V: C20.2, C4.1, D8.C, IC2.IN, L1.1, PS1.VOS, R14.2, R16.1
- new net +5V: C23.+, C6.2, D10.C, D8.A, D9.C, DISPLAY.2, IC2.OUT, IC3.IN, R22.2
- new net N$10: PS1.PG, R16.2
- new net N$13: C24.+, D9.A, IC2.ADJ, R21.2, R22.1
- new net N$14: C21.+, D11.A, IC3.ADJ, R17.2, R18.1
- new net SCL: DISPLAY.4
- new net SDA: DISPLAY.3
- net +3V3: now also C22.+, D10.A, D11.C, IC3.OUT, R18.2; no longer C5.1, C6.1, PS1.FB, PS1.VOUT
- net GND: now also C20.1, C21.-, C22.-, C23.-, C24.-, C6.1, DISPLAY.1, PS1.AGND, PS1.FSEL, PS1.MODE, R15.1, R17.1, R21.1; no longer C6.2, PS1.PGND
- net N$1: now also C3.1, PS1.SS/TR; no longer C4.1, PS1.EN, PS1.PS/SYNC, PS1.VINA
- net N$6: now also L1.2, PS1.SW; no longer L1.1, PS1.L1
- net N$7: now also PS1.FB, R14.1, R15.2; no longer L1.2, PS1.L2
- net VIN: now also C5.1, PS1.EN; no longer C3.1
Other:
- note added: "12V --> 5V"
- note added: "3.3V, 500mA"
- note added: "3V to 40V DC"
- note added: "5V --> 3V3"
- note added: "5V, 500mA"
- note added: "Audio Jack"
- note added: "Display"
- note added: "Maximum voltage: 16.8V * (2M / (0.8M + 2M)) = 12V Minimum voltage: 14V * (2M / (0.8M + 2M)) = 10V Bei 16.8V -> 3,3V = 4095 Bei 14V --> 2.75V = 3413"
- note added: "Schrittmotor"
- note added: "Schrittmotor Driver"
- note added: "Voltage Converter 14V-16.8V --> 12V"
- note added: "Vref = 1.25V"
- note removed: "Battery Voltage Converter"
- note removed: "Maximum voltage: 4.2 V * (2 M/(0.8 M+2 M)) = 3 V Maximum voltage: 3 V * (2 M/(0.8 M+2 M)) = 2,14 V Minimum voltage: 2.7 V * (2 M/(0.8 M+2 M)) = 1.93 V ADC value at 4.2 V – 12 bit setup: 3 V * (1/5) / 0.6 V * 4095 = 4095"

Commit message: beta schemaic
Parts:
- added C13, C19: (no value), rcl:C-EUC0805
- added C14, C15: 0.22u, rcl:C-EUC0805
- added C16, C18: 0.1u, rcl:C-EUC0805
- added C17: 100u, rcl:CPOL-EU085CS-1AR
- added C25: 10n, rcl:C-EUC0805
- added IC4: LM324_SOIC, IC_Linear:LM324_SOIC
- added JP1, JP2, JP3, JP4, JP5, JP6, JP7: (no value), pinhead:PINHD-1X1
- added LED_LEFT, LED_MIDDLE, LED_RIGHT: L-53GD, L-53GD:L-53GD
- added R19, R24: 5k, rcl:R-EU_R0805
- added R20, R30, R31, R32: (no value), rcl:R-EU_R0805
- added R23: 5k?, rcl:R-EU_R0805
- added R25, R26: 20, rcl:R-EU_R0805
- added R27: 10k, rcl:R-EU_R0805
- added R28: 100k, rcl:R-TRIMM3296X
- added SCHRITTMOTOR: (no value), pinhead:PINHD-1X4
- added U2: A4988SETTR-T, A4988SETTR-T:A4988SETTR-T
- C10, C11: value (none) -> 20p
- C2: value (none) -> 100n
- R1, R5: value (none) -> 500
- R2: value (none) -> 10k
- R3: value 100k -> 10k
- R4: value (none) -> 100k
Connections:
- removed net AUDIO_IN: AUDIO_JACK.TIP_2
- removed net N$15: U1.PA0_WKUP
- removed net N$17: U1.PA2
- removed net N$18: U1.PA3
- removed net N$21: U1.PA6
- removed net N$22: U1.PA7
- removed net N$24: U1.PA9
- removed net N$25: U1.PA10
- removed net N$28: U1.PA15
- removed net N$33: U1.PB0
- removed net N$34: U1.PB1
- removed net N$35: U1.PB2
- removed net N$36: U1.PB3
- removed net N$37: U1.PB4
- removed net N$38: U1.PB5
- removed net N$39: U1.PB6
- removed net N$4: AUDIO_JACK.RING_1
- removed net N$40: U1.PB7
- removed net N$41: U1.PB8
- removed net N$42: U1.PB9
- removed net N$43: U1.PB10
- removed net N$44: U1.PB11
- removed net N$45: U1.PB12
- removed net N$46: U1.PB13
- removed net N$47: U1.PB14
- removed net N$48: U1.PB15
- removed net PA11: D3.2, U1.PA11, USB-B.D-
- removed net PA12: D4.2, R13.1, U1.PA12, USB-B.D+
- removed net SCL: DISPLAY.4
- removed net SDA: DISPLAY.3
- new net DISPLAY_SCL: DISPLAY.4, U1.PB6
- new net DISPLAY_SDA: DISPLAY.3, U1.PB7
- new net DRIVER_DIR: U1.PB4, U2.DIR
- new net DRIVER_ENABLE: R23.2, U1.PA4, U2.!ENABLE
- new net DRIVER_MS1: U1.PB13, U2.MS1
- new net DRIVER_MS2: U1.PB14, U2.MS2
- new net DRIVER_MS3: U1.PB15, U2.MS3
- new net DRIVER_RESET: R19.1, U1.PA15, U2.!RESET
- new net DRIVER_SLEEP: R24.1, U1.PA5, U2.!SLEEP
- new net DRIVER_STEP: JP7.1, U1.PB3, U2.STEP
- new net LED_LEFT: LED_LEFT.A, U1.PA8
- new net LED_MIDDLE: LED_MIDDLE.A, U1.PA10
- new net LED_RIGHT: LED_RIGHT.A, U1.PA9
- new net MOTOR1A: SCHRITTMOTOR.4, U2.OUT1A
- new net MOTOR1B: SCHRITTMOTOR.3, U2.OUT1B
- new net MOTOR2A: SCHRITTMOTOR.2, U2.OUT2A
- new net MOTOR2B: SCHRITTMOTOR.1, U2.OUT2B
- new net N$26: R20.2, U2.ROSC, U2.SENSE1, U2.SENSE2
- new net N$27: C16.2, U2.VCP
- new net N$29: R25.2, USB-B.D+
- new net N$30: R26.2, USB-B.D-
- new net N$54: U2.REF
- new net N$62: C15.1, U2.VREG
- new net N$63: C18.2, U2.CP1
- new net N$64: C18.1, U2.CP2
- new net SIGNAL_IN: AUDIO_JACK.RING_1, AUDIO_JACK.TIP_2, IC4.+IN1, JP5.1
- new net SIGNAL_OPAMP: IC4.OUT1, JP6.1, R27.2, U1.PA0_WKUP
- new net USB+: D4.2, R13.1, R25.1, U1.PA12
- new net USB-: D3.2, R26.1, U1.PA11
- net +12V: now also C16.1, C17.+, JP2.1, U2.VBB1, U2.VBB2
- net +3V3: now also C14.1, C25.1, JP4.1, R19.2, R24.2, U2.VDD
- net +5V: now also IC4.V+, JP3.1
- net GND: now also C13.2, C14.2, C15.2, C17.-, C19.2, C25.2, IC4.GND, JP1.1, R20.1, R23.1, R28.A, R28.S, R30.1, R31.1, R32.1, U2.GND1, U2.GND2, U2.PAD
- net N$16: now also IC4.-IN1, R27.1, R28.E; no longer U1.PA1
- net N$19: now also LED_LEFT.C, R30.2; no longer U1.PA4
- net N$20: now also LED_RIGHT.C, R31.2; no longer U1.PA5
- net N$23: now also LED_MIDDLE.C, R32.2; no longer U1.PA8
Other:
- note added: "OPV: Vu = 1,1 - ∞"
- note added: "Voltage Converter 14V-16.8V --> 12V / 1.5A"
- note removed: "Voltage Converter 14V-16.8V --> 12V"
- moved on the sheet: AUDIO_JACK, C1, C10, C11, C8, C9, D1, D5, D6, D7, DISPLAY, LED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
