File: pcb/AutoTuner.sch (EAGLE design)
At the start: 103 parts, among them IC1 TP4054-42-SOT25-R, IC4 LM324_SOIC, Q1 32,768kHz, Q2 BSS123, Q3 BSS84, U1 STM32F103C8T6, U2 A4988SETTR-T, U3 AMS1117-3.3, U4 AMS1117-5.0, Y1 8MHz

Commit message: schematic beta 1
Parts:
- added BATTERIE: (no value), pinhead:PINHD-1X2
Connections:
- net +3V3: no longer R13.2
- net +5V: now also R13.2
- net GND: now also BATTERIE.1, X1-1.KL; no longer X1-2.KL
- net N$15: now also X1-2.KL; no longer X1-1.KL
- net VBAT: now also BATTERIE.2
Other:
- note added: "Batterie"
- moved on the sheet: C13, C19, C25, C26, D12, D13, U1
