File: pcb/AutoTunerV1.sch (EAGLE design)
At the start: 104 parts, among them IC1 TP4054-42-SOT25-R, IC4 LM324_SOIC, Q1 32,768kHz, Q2 BSS123, Q3 BSS84, U1 STM32F103C8T6, U2 A4988SETTR-T, U3 AMS1117-3.3, U4 AMS1117-5.0, Y1 8MHz

Commit message: board v1 release
Parts:
- removed C13, C19, C25: 10n, rcl:C-EUC0805
- removed C14, C15: 0.22u, rcl:C-EUC0805
- removed C16, C18: 0.1u, rcl:C-EUC0805
- removed C17: 100u, rcl:CPOL-EU085CS-1AR
- removed C20, C6: (no value), rcl:C-EUC0805
- removed C27: 100n, rcl:C-EUC0805
- removed D12: 1N4004, diode:1N4004
- removed D13: TESD5V0L1UC_RJG, TESD5V0L1UC_RJG:TESD5V0L1UC_RJG
- removed JP1, JP2, JP3, JP4, JP5, JP6, JP7: (no value), pinhead:PINHD-1X1
- removed PS1: TPS62147RGXR, TPS62147RGXR:TPS62147RGXR
- removed R15, R16: 100k, rcl:R-EU_R0805
- removed R19, R24: 5k, rcl:R-EU_R0805
- removed R20: (no value), rcl:R-EU_R0805
- removed R23: 5k?, rcl:R-EU_R0805
- removed R28: 100k, rcl:R-TRIMM3296X
- removed SCHRITTMOTOR: (no value), pinhead:PINHD-1X4
- removed X1: (no value), con-ptr500:AK300/2
- added D8, D9: 1N4004, diode:1N4004
- added DC-MOTOR: 22-27-2021-02, con-molex:22-27-2021-02
- added TP1, TP3, TP4, TP5, TP6: TPB1,27, testpad:TPB1,27
- BATTERIE: value (none) -> 22-27-2021-02; device pinhead:PINHD-1X2 -> con-molex:22-27-2021-02
- C3: value 2.2nF -> 22u
- C4: value 47uF -> 10-100uF; device rcl:C-EUC0805 -> rcl:CPOL-EUB45181A
- C5: value 10uF -> 22u
- D2, D3, D4, D5, D6: LCSC_PART (none) -> C7420372
- L1: value 1.5uH -> 4.7u; device PSPCAQ54:PSPCAQ54 -> DFE252012P-4R7M=P2:DFE252012P-4R7M=P2; LCSC_PART C2686105 -> C391306
- Q3: LCSC_PARTS (none) -> C10487
- R10: value 25k -> 2M
- R11: value (none) -> 100k
- R13: value 1k5 -> 1k5 / 4k7
- R14: value 1.62M -> 100k; device rcl:R-EU_R0805 -> rcl:R-TRIMM43P
- R9: value 100k -> 800k
- U2: value A4988SETTR-T -> TPS613222ADBVR; device A4988SETTR-T:A4988SETTR-T -> TPS613222ADBVR:TPS613222ADBVR; LCSC_PART (none) -> C2071163
- U4: value AMS1117-5.0 -> BD6222HFP-TRHRP7_ROM-M; device AMS1117-5.0:AMS1117-5.0 -> H-Brücke_BD622HFP-TR02:BD6222HFP-TRHRP7_ROM-M; LCSC_PART C6187 -> (none)
- renumbered S1 to SELECT, S3 to RIGHT, S4 to LEFT
Connections:
- net A_BATTERY_LEVEL renamed BATTERY_LEVEL
- removed net +12V: C16.1, C17.+, C4.1, C6.2, JP2.1, L1.1, PS1.VOS, R14.2, R16.1, U2.VBB1, U2.VBB2, U4.VIN
- removed net DRIVER_DIR: U1.PB4, U2.DIR
- removed net DRIVER_ENABLE: R23.2, U1.PA4, U2.!ENABLE
- removed net DRIVER_MS1: U1.PB13, U2.MS1
- removed net DRIVER_MS2: U1.PB14, U2.MS2
- removed net DRIVER_MS3: U1.PB15, U2.MS3
- removed net DRIVER_RESET: R19.1, U1.PA15, U2.!RESET
- removed net DRIVER_SLEEP: R24.1, U1.PA5, U2.!SLEEP
- removed net DRIVER_STEP: JP7.1, U1.PB3, U2.STEP
- removed net MOTOR1A: SCHRITTMOTOR.4, U2.OUT1A
- removed net MOTOR1B: SCHRITTMOTOR.3, U2.OUT1B
- removed net MOTOR2A: SCHRITTMOTOR.2, U2.OUT2A
- removed net MOTOR2B: SCHRITTMOTOR.1, U2.OUT2B
- removed net N$10: PS1.PG, R16.2
- removed net N$15: C27.1, D12.A, D13.2, X1-2.KL
- removed net N$26: R20.2, U2.ROSC, U2.SENSE1, U2.SENSE2
- removed net N$27: C16.2, U2.VCP
- removed net N$54: U2.REF
- removed net N$62: C15.1, U2.VREG
- removed net N$63: C18.2, U2.CP1
- removed net N$64: C18.1, U2.CP2
- removed net VKLEMME: D1.A, D12.C, IC1.VCC, Q3.G, R11.2, R7.1, R8.1
- new net MOTORA: DC-MOTOR-2.S, U4.OUT1
- new net MOTORB: DC-MOTOR-1.S, U4.OUT2
- new net MOTOR_PWM1: D8.A, U1.PB0
- new net MOTOR_PWM2: D9.A, U1.PB1
- new net N$14: D9.C, U4.RIN
- new net PAD: U4.EPAD
- new net VBUS: C12.1, D1.A, D2.2, IC1.VCC, Q3.G, R11.2, R7.1, R8.1, USB-B.VCC
- net +3V3: now also IC4.V+, TP4.TP; no longer C13.1, C14.1, C19.1, C25.1, JP4.1, R19.2, R24.2, U2.VDD
- net +5V: now also C3.2, TP3.TP, U2.VOUT; no longer C12.1, C20.2, D2.2, IC4.V+, JP3.1, U4.VOUT, USB-B.VCC
- net BUTTON_1: now also U1.PB13; no longer U1.PB11
- net BUTTON_2: now also U1.PB14; no longer U1.PB0
- net BUTTON_3: now also U1.PB15; no longer U1.PB1
- net GND: now also BATTERIE-1.S, C3.1, C4.-, C5.1, R14.A, R14.S, TP1.TP, U2.GND, U4.GND; no longer BATTERIE.1, C13.2, C14.2, C15.2, C17.-, C19.2, C20.1, C25.2, C27.2, C3.2, C4.2, C5.2, C6.1, D13.1, JP1.1, PS1.AGND, PS1.FSEL, PS1.GND, PS1.MODE, R15.1, R20.1, R23.1, R28.A, R28.S, U2.GND1, U2.GND2, U2.PAD, U4.GND/ADJ, X1-1.KL
- net LED_MIDDLE: now also U1.PA9; no longer U1.PA10
- net LED_RIGHT: now also U1.PA10; no longer U1.PA9
- net N$1: now also L1.2, U2.SW; no longer C3.1, PS1.SS/TR
- net N$16: now also IC4.-IN2, R14.E; no longer IC4.-IN1, R28.E
- net N$6: now also D8.C, U4.FIN; no longer L1.2, PS1.SW
- net N$7: now also U4.VCC; no longer PS1.FB, R14.1, R15.2
- net SIGNAL_IN: now also IC4.+IN2, TP5.TP; no longer IC4.+IN1, JP5.1
- net SIGNAL_OPAMP: now also IC4.OUT2, TP6.TP, U1.PA1; no longer IC4.OUT1, JP6.1, U1.PA0_WKUP
- net VBAT: now also BATTERIE-2.S, C4.+, U4.VREF; no longer BATTERIE.2
- net VIN: now also C5.2, L1.1; no longer C5.1, PS1.EN, PS1.VIN
Other:
- note added: "32kHz Quarz ok"
- note added: "5V --> 3V3 ok"
- note added: "8MHz Quarz ok"
- note added: "Audio Jack ok"
- note added: "Batterie ok"
- note added: "Battery charger ok"
- note added: "DC - Motor ok"
- note added: "DC MOTOR H-Bridge ok"
- note added: "Maximum voltage: 4.2V * (2M / (0.8M + 2M)) = Minimum voltage: 3.0V * (2M / (0.8M + 2M)) ="
- note added: "OPV: Vu = 1,1 - ∞ok"
- note added: "Power IN ok"
- note added: "STM32"
- note added: "Voltage Boost Converter ok"
- note added: "Voltage Source Selection ok"
- note removed: "12V --> 5V"
- note removed: "32kHz Quarz"
- note removed: "5V --> 3V3"
- note removed: "8MHz Quarz"
- note removed: "Audio Jack"
- note removed: "Batterie"
- note removed: "Battery charger"
- note removed: "Maximum voltage: 16.8V * (2M / (0.8M + 2M)) = 12V Minimum voltage: 14V * (2M / (0.8M + 2M)) = 10V Bei 16.8V -> 3,3V = 4095 Bei 14V --> 2.75V = 3413"
- note removed: "OPV: Vu = 1,1 - ∞"
- note removed: "Power IN"
- note removed: "Schrittmotor"
- note removed: "Schrittmotor Driver"
- note removed: "Voltage Converter 14V-16.8V --> 12V / 1.5A"
- note removed: "Voltage Source Selection"
