File: pcb/AutoTunerV2.sch (EAGLE design)
At the start: 82 parts, among them IC1 TP4054-42-SOT25-R, IC4 LM324_SOIC, Q1 32,768kHz, Q2 BSS123, Q3 BSS84, U1 STM32F103C8T6, U2 TPS613222ADBVR, U3 AMS1117-3.3, U4 BD6222HFP-TRHRP7_ROM-M, Y1 8MHz

Commit message: board v2 release
Parts:
- removed D5, D6, D7: TESD5V0L1UC_RJG, TESD5V0L1UC_RJG:TESD5V0L1UC_RJG
- removed TP1, TP3, TP4, TP5, TP6: TPB1,27, testpad:TPB1,27
- removed U3: AMS1117-3.3, AMS1117-3.3:AMS1117-3.3
- added C13, C14, C6: 10n, rcl:C-EUC0805
- added C15: 120p, rcl:C-EUC0805
- added IC2: 317EMP, linear:317EMP
- added R15: 5, rcl:R-EU_R0805
- added SCHOTTKYDIODE0805: (no value), rcl:C-USC0805
- R14: device rcl:R-TRIMM43P -> rcl:R-TRIMM64Y
Connections:
- new net N$10: C15.1, R15.1
- net +3V3: now also C13.1, C14.1, C6.1, IC2.VO; no longer D5.2, TP4.TP, U3.VOUT
- net +5V: now also C15.2, IC2.VI, SCHOTTKYDIODE0805.2; no longer R13.2, TP3.TP, U3.VIN
- net GND: now also C13.2, C14.2, C6.2, IC2.ADJ, R14.E; no longer D5.1, D6.1, D7.1, R14.A, TP1.TP, U3.GND/ADJ
- net N$1: now also R15.2, SCHOTTKYDIODE0805.1
- net N$16: now also IC4.-IN3, R14.A, R27.2; no longer IC4.-IN2, R14.E, R27.1
- net SIGNAL_IN: now also IC4.+IN3; no longer IC4.+IN2, TP5.TP
- net SIGNAL_OPAMP: now also IC4.OUT3, R27.1; no longer IC4.OUT2, R27.2, TP6.TP
- net SWDCLK: no longer D7.2
- net SWDIO: no longer D6.2
- net VBUS: now also R13.2
Other:
- moved on the sheet: C1, C21, C22, C3, C4, C5, D8, D9, IC4, L1, LED, POWER_LED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

Commit message: board v2 release 2.0
Parts:
- removed C21, C22: (no value), rcl:C-EUC0805
- removed C3, C5: 22u, rcl:C-EUC0805
- added C16, C17, C18, C19: 22u, rcl:C-EUC1206
- added R16, R17, R18: 0, rcl:R-EU_R0805
- LED1, POWER_LED: LCSC_PART (none) -> C2297
- LED2, RED_LED: LCSC_PART (none) -> C84256
- R1, R5: value 500 -> 68
- R13: value 1k5 / 4k7 -> 1k5
- R15: value 5 -> 5R
- R30, R31, R32: value (none) -> 100
- renumbered LED to RED_LED
Connections:
- new net N$13: C18.1, IC2.VO, R17.1
- new net N$45: R18.2, U1.PA1
- net +3V3: now also R13.2, R17.2; no longer C21.2, IC2.VO
- net +5V: now also C19.1, R16.2; no longer C15.2, C22.2, C3.2, SCHOTTKYDIODE0805.2, U2.VOUT
- net GND: now also C16.2, C17.2, C18.2, C19.2; no longer C21.1, C22.1, C3.1, C5.1
- net N$7: now also C15.2, C17.1, R16.1, SCHOTTKYDIODE0805.2, U2.VOUT; no longer U4.VCC
- net SIGNAL_OPAMP: now also R18.1; no longer U1.PA1
- net VBAT: now also U4.VCC
- net VBUS: no longer R13.2
- net VIN: now also C16.1; no longer C5.2
Other:
- moved on the sheet: IC4, R14, R27

Commit message: board v2 main release & oder
Parts:
- removed D1: MBR0520LT1G, Diode:SCHOTTKY_MBR0520LT1GDO-219
- removed SCHOTTKYDIODE0805: (no value), rcl:C-USC0805
- added R19: 6k8, rcl:R-EU_R0805
- added R20: 330k, rcl:R-EU_R0805
- added R21: 470k, rcl:R-EU_R0805
- added SCHOTTKY, SCHOTTKY1: (no value), diode:DIODE-SOD323-R
- C4: value 10-100uF -> 100uF
- L1: LCSC_PART C391306 -> C3093670
- R1, R5: LCSC_PART (none) -> C17802
- R10: value 2M -> 1M
- R6: value 1k66 -> 2k2
- R9: value 800k -> 1M
- renumbered IC1 to BATTERYCHARGER, IC4 to OPV, R14 to TRIMMER, S2 to BOOT, U1 to STM32, U2 to DCDC, U4 to H-BRUECKE
Connections:
- new net N$46: R20.2, R21.1
- new net N$47: R10.2, R20.1, R29.1
- net GND: now also R19.1, R9.1; no longer R10.1
- net N$1: now also SCHOTTKY.A; no longer SCHOTTKYDIODE0805.1
- net N$4: now also R10.1, R9.2; no longer R10.2, R29.1, R9.1
- net N$7: now also SCHOTTKY.C; no longer SCHOTTKYDIODE0805.2
- net N$8: now also R19.2
- net VBAT: now also R21.2; no longer R9.2
- net VBUS: now also SCHOTTKY1.A; no longer D1.A
- net VIN: now also SCHOTTKY1.C; no longer D1.C
Other:
- moved on the sheet: C18, C19, C7, IC2, R10, R17, R29, R9
