File: pcb/v3/AutoTunerV3.brd (EAGLE design)
At the start: 100 x 90 mm, 95 parts, among them IC1 317EMP, IC2 317EMP, Q1 32,768kHz, Q2 BSS123, Q3 BSS84, Y1 8MHz

Commit message: frequency calcs
Parts:
- removed BATTERIE, DC-MOTOR: (no value), con-molex:6410-02
- removed IC1: 317EMP, linear:SOT223
- added +3V3, +5V, SIGNAL_IN, SIGNAL_OPAMP, VBAT, VBUS: TPB1,27, testpad:B1,27
- added BATTERIE1, BATTERIE2, MOTOR: (no value), con-molex:6410-02
- added BUZZER: AL11P, buzzer:AL11P
- added C16: 100n, rcl:C0805
- added C17: 47u, rcl:C0805
- added L1: 1.5u, XFL4020-152MEC:IND_XFL4020-152MEC
- added R28, R34, R41: 10k, rcl:R0805
- added R38, R39: 100k, rcl:R0805
- added R40: 523k, rcl:R0805
- added T1: (no value), transistor:SOT23-EBC
- added U1: TPS63070RNMR, TPS63070RNMR:VREG_TPS63070RNMR
- C3: value 22u -> 10u; device rcl:C1206 -> rcl:C0805
- C4: value 100uF -> 100u; device rcl:B45181A -> rcl:E2,5-6E
- C5: value 22u -> 47u; device rcl:C1206 -> rcl:C0805
- JP2, ST_LINK: device pinhead:1X04 -> pinhead:1X04/90
- moved C15 138.5 mm to (80.3, 11.1)
- moved R16 130.5 mm to (74.6, 11.1)
- moved JP1 116.3 mm to (83.2, 5.43), turned to 270 degrees
- moved R15 111.1 mm to (2.84, 68.4)
- moved TRIMMER 109.5 mm to (77.2, 5.43), turned to 180 degrees
- moved C3 105.4 mm to (23.4, 58.9), turned to 180 degrees
- moved C5 104.8 mm to (23.4, 61.1), turned to 180 degrees
- moved GND 80.4 mm to (5.70, 68.4)
- moved POWER_LED 44.0 mm to (96.5, 50.2), turned to 90 degrees
- moved R1 43.7 mm to (96.5, 48.3)
- moved LED1 34.7 mm to (9.27, 53.2)
- moved Q2 34.0 mm to (12.4, 52.3)
- moved LED2 33.4 mm to (5.46, 52.0)
- moved R19 32.5 mm to (14.3, 48.1)
- moved R6 32.5 mm to (12.1, 48.1)
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Connections:
- removed net N$3: POWER_LED.C, R1.1
- new net BUZZER: R28.1, STM32.45
- new net N$1: POWER_LED.A, R1.2
- new net N$53: BATTERIE1.1, R15.2
- new net N$54: BUZZER.+, T1.C
- new net N$55: BUZZER.-, R34.1
- new net N$56: R28.2, T1.B
- new net N$58: L1.2, U1.9
- new net N$59: L1.1, U1.11
- new net N$60: C16.1, U1.3
- new net N$61: R38.1, U1.2
- new net N$62: R39.2, R40.1, U1.5
- new net N$64: R41.2, U1.14
- net +3V3: now also +3V3.TP, R1.1; no longer POWER_LED.A
- net +5V: now also +5V.TP, C3.1, C5.1, R34.2, R38.2, R40.2, U1.7_8; no longer R15.2
- net GND: now also AUDIO_JACK.3, AUDIO_JACK.4, BATTERIE2.1, C16.2, C17.2, POWER_LED.C, R39.1, RED_LED.C, T1.E, U1.10, U1.15, U1.4, U1.6; no longer BATTERIE.1, IC1.1, R1.2, R5.1
- net MOTORA: now also MOTOR.2; no longer DC-MOTOR.2
- net MOTORB: now also MOTOR.1; no longer DC-MOTOR.1
- net N$2: now also R5.1, RED_LED.A; no longer R5.2, RED_LED.C
- net N$45: now also STM32.12; no longer STM32.11
- net N$51: now also BATTERIE2.2; no longer C3.1, IC1.4
- net PC13: now also R5.2; no longer RED_LED.A
- net SIGNAL_IN: now also SIGNAL_IN.TP
- net SIGNAL_OPAMP: now also SIGNAL_OPAMP.TP
- net VBAT: now also BATTERIE1.2, VBAT.TP; no longer BATTERIE.2
- net VBUS: now also VBUS.TP
- net VIN: now also C17.1, R41.1, U1.1, U1.12_13; no longer C5.1, IC1.3
Routing:
- net DISPLAY_SCL: track 0.00 -> 69.1 mm, vias 0 -> 1
- net DISPLAY_SDA: track 0.00 -> 61.7 mm, vias 0 -> 1
- net GND: track 285.8 -> 325.5 mm, vias 10 -> 16
- net BUZZER: track 0.00 -> 35.3 mm
- net VBAT: track 129.2 -> 96.3 mm, vias 1 -> 2
- net RESET: track 10.6 -> 35.8 mm, vias 0 -> 2
- net N$45: track 77.5 -> 53.1 mm
- net SWDCLK: track 0.00 -> 24.3 mm
- net +5V: track 2.54 -> 26.8 mm
- net +3V3: track 147.2 -> 170.2 mm, vias 7 -> 6
- net SWDIO: track 0.00 -> 22.5 mm
- net N$39: track 8.43 -> 27.6 mm
- net N$48: track 8.49 -> 25.4 mm, vias 0 -> 1
- net BOOT0: track 0.00 -> 16.2 mm, vias 0 -> 2
- net N$49: track 8.60 -> 22.5 mm, vias 0 -> 1
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- added copper zone on layer 1, net +5V
- removed copper zone on layer 1, net N$1
- removed copper zone on layer 1, net N$10
- removed copper zone on layer 1, net N$7
Other:
- board size 100 x 90 mm -> 100 x 80 mm
- board text added: "-"
- board text added: "Battery 1"
- board text added: "Battery 2"
- board text added: "Buzzer"
- board text added: "Gabriel Unterweger AutoTuner - 5BEL - V3"
- board text added: "MOTOR"
- board text added: "PC13"
- board text added: "Power"
- board text added: "ST-Link"
- board text added: "uC"
- board text removed: "Gabriel Unterweger AutoTuner - 5BEL - V1"
