File: pcb/v3/AutoTunerV3.sch (EAGLE design)
At the start: 95 parts, among them IC1 317EMP, IC2 317EMP, Q1 32,768kHz, Q2 BSS123, Q3 BSS84, Y1 8MHz

Commit message: frequency calcs
Parts:
- removed BATTERIE, DC-MOTOR: 22-27-2021-02, con-molex:22-27-2021-02
- removed IC1: 317EMP, linear:317EMP
- added +3V3, +5V, SIGNAL_IN, SIGNAL_OPAMP, VBAT, VBUS: TPB1,27, testpad:TPB1,27
- added BATTERIE1, BATTERIE2, MOTOR: 22-27-2021-02, con-molex:22-27-2021-02
- added BUZZER: AL11P, buzzer:AL11P
- added C16: 100n, rcl:C-EUC0805
- added C17: 47u, rcl:C-EUC0805
- added L1: 1.5u, XFL4020-152MEC:XFL4020-152MEC
- added R28, R34, R41: 10k, rcl:R-EU_R0805
- added R38, R39: 100k, rcl:R-EU_R0805
- added R40: 523k, rcl:R-EU_R0805
- added T1: (no value), transistor:-NPN-SOT23-EBC
- added U1: TPS63070RNMR, TPS63070RNMR:TPS63070RNMR
- C3: value 22u -> 10u; device rcl:C-EUC1206 -> rcl:C-EUC0805; LCSC_PART C5672 -> (none)
- C4: value 100uF -> 100u; device rcl:CPOL-EUB45181A -> rcl:CPOL-EUE2,5-6E
- C5: value 22u -> 47u; device rcl:C-EUC1206 -> rcl:C-EUC0805; LCSC_PART C5672 -> (none)
- JP2, ST_LINK: device pinhead:PINHD-1X4 -> pinhead:PINHD-1X4/90
Connections:
- removed net N$3: POWER_LED.C, R1.1
- new net BUZZER: R28.1, STM32.PB8
- new net N$1: POWER_LED.A, R1.2
- new net N$53: BATTERIE1-1.S, R15.2
- new net N$54: BUZZER.2, T1.C
- new net N$55: BUZZER.1, R34.1
- new net N$56: R28.2, T1.B
- new net N$58: L1.2, U1.L2
- new net N$59: L1.1, U1.L1
- new net N$60: C16.1, U1.VAUX
- new net N$61: R38.1, U1.PG
- new net N$62: R39.2, R40.1, U1.FB
- new net N$64: R41.2, U1.EN
- net +3V3: now also +3V3.TP, R1.1; no longer POWER_LED.A
- net +5V: now also +5V.TP, C3.1, C5.1, R34.2, R38.2, R40.2, U1.VOUT; no longer R15.2
- net GND: now also AUDIO_JACK.RING_2, AUDIO_JACK.TIP_1, BATTERIE2-1.S, C16.2, C17.2, POWER_LED.C, R39.1, RED_LED.C, T1.E, U1.FB2, U1.GND, U1.PGND, U1.VSEL; no longer BATTERIE-1.S, IC1.ADJ, R1.2, R5.1
- net MOTORA: now also MOTOR-2.S; no longer DC-MOTOR-2.S
- net MOTORB: now also MOTOR-1.S; no longer DC-MOTOR-1.S
- net N$2: now also R5.1, RED_LED.A; no longer R5.2, RED_LED.C
- net N$45: now also STM32.PA2; no longer STM32.PA1
- net N$51: now also BATTERIE2-2.S; no longer C3.1, IC1.VO
- net PC13: now also R5.2; no longer RED_LED.A
- net SIGNAL_IN: now also SIGNAL_IN.TP
- net SIGNAL_OPAMP: now also SIGNAL_OPAMP.TP
- net VBAT: now also BATTERIE1-2.S, VBAT.TP; no longer BATTERIE-2.S
- net VBUS: now also VBUS.TP
- net VIN: now also C17.1, R41.1, U1.PS/SYNC, U1.VIN; no longer C5.1, IC1.VI
Other:
- note added: "Buzzer"
- moved on the sheet: C3, C5, GND, JP1, JP2, LED3, LED4, LED5, LED6, LED_LEFT, LED_MIDDLE, LED_RIGHT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
