File: pcb/v2/AutoTunerV2.sch (EAGLE design)
At the start: 86 parts, among them IC2 317EMP, Q1 32,768kHz, Q2-N7000 BSS123, Q3 BSS84, Y1 8MHz

Commit message: doku
Other:
- note added: "5V --> 3V3"
- note added: "Audio Jack"
- note added: "Batterie"
- note added: "Battery charger"
- note added: "DC - Motor"
- note added: "DC MOTOR H-Bridge"
- note added: "OPV: Vu = 1,1 - ∞"
- note added: "Power IN"
- note added: "Voltage Boost Converter"
- note added: "Voltage Source Selection"
- note removed: "5V --> 3V3 ok"
- note removed: "Audio Jack ok"
- note removed: "Batterie ok"
- note removed: "Battery charger ok"
- note removed: "DC - Motor ok"
- note removed: "DC MOTOR H-Bridge ok"
- note removed: "Maximum voltage: 4.2V * (2M / (0.8M + 2M)) = Minimum voltage: 3.0V * (2M / (0.8M + 2M)) ="
- note removed: "OPV: Vu = 1,1 - ∞ok"
- note removed: "Power IN ok"
- note removed: "Test Points"
- note removed: "Voltage Boost Converter ok"
- note removed: "Voltage Source Selection ok"
- moved on the sheet: AUDIO_JACK, C7, DC-MOTOR-1, DC-MOTOR-2, LED_LEFT, LED_MIDDLE, LED_RIGHT, R10, R20, R21, R29, R30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
